Commit message: 整理了xacro文件,规范命名

File: src/robot_description/urdf/robot.custom.xacro (robot description, xacro)
@@ -1,185 +1,8 @@
 <?xml version="1.0"?>
 <robot name="four_wheel_robot" xmlns:xacro="http://www.ros.org/wiki/xacro">
-  <!-- 机器人常量 -->
-  <xacro:property name="PI" value="3.1415926535897931"/>
-  <!-- 底盘属性 -->
-  <xacro:property name="chassis_length" value="0.300"/>
-  <xacro:property name="chassis_width" value="0.200"/>
-  <xacro:property name="chassis_height" value="0.050"/>
-  <xacro:property name="chassis_mass" value="5.0"/>
-  <!-- 轮子属性 -->
-  <xacro:property name="wheel_radius" value="0.030"/>
-  <xacro:property name="wheel_thickness" value="0.025"/>
-  <xacro:property name="wheel_mass" value="0.5"/>
-  <!-- 安装位置偏移 -->
-  <xacro:property name="wheel_z_offset" value="0.030"/>
-  <xacro:property name="wheel_x_offset" value="0.100"/>
-  <!-- 底盘链接 (参考坐标系) -->
-  <link name="base_link">
-    <visual>
-      <origin xyz="0 0 0" rpy="0 0 0"/>
-      <geometry>
-        <box size="${chassis_length} ${chassis_width} ${chassis_height}"/>
-      </geometry>
-      <material name="grey">
-        <color rgba="0.5 0.5 0.5 1.0"/>
-      </material>
-    </visual>
-    <collision>
-      <origin xyz="0 0 0" rpy="0 0 0"/>
-      <geometry>
-        <box size="${chassis_length} ${chassis_width} ${chassis_height}"/>
-      </geometry>
-    </collision>
-    <inertial>
-      <origin xyz="0 0 0" rpy="0 0 0"/>
-      <mass value="${chassis_mass}"/>
-      <inertia ixx="${chassis_mass / 12.0 * (chassis_width**2 + chassis_height**2)}"
-               ixy="0" ixz="0"
-               iyy="${chassis_mass / 12.0 * (chassis_length**2 + chassis_height**2)}"
-               iyz="0"
-               izz="${chassis_mass / 12.0 * (chassis_length**2 + chassis_width**2)}"/>
-    </inertial>
-  </link>
-  <link name="base_footprint" />
-  <joint name="base_joint" type="fixed">
-    <parent link="base_footprint" />
-    <child link="base_link" />
-    <origin xyz="0.0 0.0 ${wheel_z_offset + wheel_radius - 0.001}" rpy="0 0 0" />
-  </joint>
-  <!-- 左前轮 -->
-  <link name="front_left_wheel">
-    <visual>
-      <origin xyz="0 0 0" rpy="${PI/2} 0 0"/>
-      <geometry>
-        <cylinder radius="${wheel_radius}" length="${wheel_thickness}"/>
-      </geometry>
-      <material name="black">
-        <color rgba="0.1 0.1 0.1 1.0"/>
-      </material>
-    </visual>
-    <collision>
-      <origin xyz="0 0 0" rpy="${PI/2} 0 0"/>
-      <geometry>
-        <cylinder radius="${wheel_radius}" length="${wheel_thickness}"/>
-      </geometry>
-    </collision>
-    <inertial>
-      <origin xyz="0 0 0" rpy="0 0 0"/>
-      <mass value="${wheel_mass}"/>
-      <inertia ixx="${wheel_mass / 12.0 * (3*wheel_radius**2 + wheel_thickness**2)}"
-               ixy="0" ixz="0"
-               iyy="${wheel_mass / 12.0 * (3*wheel_radius**2 + wheel_thickness**2)}"
-               iyz="0"
-               izz="${wheel_mass / 2.0 * wheel_radius**2}"/>
-    </inertial>
-  </link>
-  <joint name="front_left_wheel_joint" type="continuous">
-    <parent link="base_link"/>
-    <child link="front_left_wheel"/>
-    <origin xyz="${wheel_x_offset} ${chassis_width/2 + wheel_thickness/2} ${-wheel_z_offset}" rpy="0 0 0"/>
-    <axis xyz="0 1 0"/>
-  </joint>
-  <!-- 右前轮 -->
-  <link name="front_right_wheel">
-    <visual>
-      <origin xyz="0 0 0" rpy="${PI/2} 0 0"/>
-      <geometry>
-        <cylinder radius="${wheel_radius}" length="${wheel_thickness}"/>
-      </geometry>
-      <material name="black">
-        <color rgba="0.1 0.1 0.1 1.0"/>
-      </material>
-    </visual>
-    <collision>
-      <origin xyz="0 0 0" rpy="${PI/2} 0 0"/>
-      <geometry>
-        <cylinder radius="${wheel_radius}" length="${wheel_thickness}"/>
-      </geometry>
-    </collision>
-    <inertial>
-      <origin xyz="0 0 0" rpy="0 0 0"/>
-      <mass value="${wheel_mass}"/>
-      <inertia ixx="${wheel_mass / 12.0 * (3*wheel_radius**2 + wheel_thickness**2)}"
-               ixy="0" ixz="0"
-               iyy="${wheel_mass / 12.0 * (3*wheel_radius**2 + wheel_thickness**2)}"
-               iyz="0"
-               izz="${wheel_mass / 2.0 * wheel_radius**2}"/>
-    </inertial>
-  </link>
-  <joint name="front_right_wheel_joint" type="continuous">
-    <parent link="base_link"/>
-    <child link="front_right_wheel"/>
-    <origin xyz="${wheel_x_offset} ${-chassis_width/2 - wheel_thickness/2} ${-wheel_z_offset}" rpy="0 0 0"/>
-    <axis xyz="0 1 0"/>
-  </joint>
-  <!-- 左后轮 -->
-  <link name="rear_left_wheel">
-    <visual>
-      <origin xyz="0 0 0" rpy="${PI/2} 0 0"/>
-      <geometry>
-        <cylinder radius="${wheel_radius}" length="${wheel_thickness}"/>
-      </geometry>
-      <material name="black">
-        <color rgba="0.1 0.1 0.1 1.0"/>
-      </material>
-    </visual>
-    <collision>
-      <origin xyz="0 0 0" rpy="${PI/2} 0 0"/>
-      <geometry>
-        <cylinder radius="${wheel_radius}" length="${wheel_thickness}"/>
-      </geometry>
-    </collision>
-    <inertial>
-      <origin xyz="0 0 0" rpy="0 0 0"/>
-      <mass value="${wheel_mass}"/>
-      <inertia ixx="${wheel_mass / 12.0 * (3*wheel_radius**2 + wheel_thickness**2)}"
-               ixy="0" ixz="0"
-               iyy="${wheel_mass / 12.0 * (3*wheel_radius**2 + wheel_thickness**2)}"
-               iyz="0"
-               izz="${wheel_mass / 2.0 * wheel_radius**2}"/>
-    </inertial>
-  </link>
-  <joint name="rear_left_wheel_joint" type="continuous">
-    <parent link="base_link"/>
-    <child link="rear_left_wheel"/>
-    <origin xyz="${-wheel_x_offset} ${chassis_width/2 + wheel_thickness/2} ${-wheel_z_offset}" rpy="0 0 0"/>
-    <axis xyz="0 1 0"/>
-  </joint>
-  <!-- 右后轮 -->
-  <link name="rear_right_wheel">
-    <visual>
-      <origin xyz="0 0 0" rpy="${PI/2} 0 0"/>
-      <geometry>
-        <cylinder radius="${wheel_radius}" length="${wheel_thickness}"/>
-      </geometry>
-      <material name="black">
-        <color rgba="0.1 0.1 0.1 1.0"/>
-      </material>
-    </visual>
-    <collision>
-      <origin xyz="0 0 0" rpy="${PI/2} 0 0"/>
-      <geometry>
-        <cylinder radius="${wheel_radius}" length="${wheel_thickness}"/>
-      </geometry>
-    </collision>
-    <inertial>
-      <origin xyz="0 0 0" rpy="0 0 0"/>
-      <mass value="${wheel_mass}"/>
-      <inertia ixx="${wheel_mass / 12.0 * (3*wheel_radius**2 + wheel_thickness**2)}"
-               ixy="0" ixz="0"
-               iyy="${wheel_mass / 12.0 * (3*wheel_radius**2 + wheel_thickness**2)}"
-               iyz="0"
-               izz="${wheel_mass / 2.0 * wheel_radius**2}"/>
-    </inertial>
-  </link>
-  <joint name="rear_right_wheel_joint" type="continuous">
-    <parent link="base_link"/>
-    <child link="rear_right_wheel"/>
-    <origin xyz="${-wheel_x_offset} ${-chassis_width/2 - wheel_thickness/2} ${-wheel_z_offset}" rpy="0 0 0"/>
-    <axis xyz="0 1 0"/>
-  </joint>
+  <!-- 共享模型定义 -->
+  <xacro:include filename="$(find robot_description)/urdf/robot.model.xacro" />
   <!-- Custom ros2_control hardware interface -->
-  <xacro:include filename="$(find robot_description)/urdf/robot.custom_control.xacro" />
+  <xacro:include filename="$(find robot_description)/urdf/control/custom.control.xacro" />
   <xacro:robot_custom_ros2_control />
 </robot>

File: src/robot_description/urdf/robot.model.xacro (robot description, xacro)
@@ -1,4 +1,5 @@
 <?xml version="1.0"?>
-<robot name="four_wheel_robot" xmlns:xacro="http://www.ros.org/wiki/xacro">
+<robot xmlns:xacro="http://www.ros.org/wiki/xacro">
+  <!-- ========== 公共属性 ========== -->
   <!-- 机器人常量 -->
   <xacro:property name="PI" value="3.1415926535897931"/>
@@ -15,8 +16,5 @@
   <xacro:property name="wheel_z_offset" value="0.030"/>
   <xacro:property name="wheel_x_offset" value="0.100"/>
-  <!-- Gazebo 材质 (放在 link 定义之前) -->
-  <gazebo reference="base_link">
-    <material>Gazebo/Grey</material>
-  </gazebo>
+  <!-- ========== 底盘 ========== -->
   <!-- 底盘链接 (参考坐标系) -->
   <link name="base_link">
@@ -48,12 +46,9 @@
   <link name="base_footprint" />
   <joint name="base_joint" type="fixed">
-            <parent link="base_footprint" />
-            <child link="base_link" />
-            <origin xyz="0.0 0.0 ${wheel_z_offset + wheel_radius - 0.001}" rpy="0 0 0" />
+    <parent link="base_footprint" />
+    <child link="base_link" />
+    <origin xyz="0.0 0.0 ${wheel_z_offset + wheel_radius - 0.001}" rpy="0 0 0" />
   </joint>
-  <!-- Gazebo 材质 - 左前轮 -->
-  <gazebo reference="front_left_wheel">
-    <material>Gazebo/Black</material>
-  </gazebo>
+  <!-- ========== 轮子 ========== -->
   <!-- 左前轮 -->
   <link name="front_left_wheel">
@@ -89,8 +84,4 @@
     <axis xyz="0 1 0"/>
   </joint>
-  <!-- Gazebo 材质 - 右前轮 -->
-  <gazebo reference="front_right_wheel">
-    <material>Gazebo/Black</material>
-  </gazebo>
   <!-- 右前轮 -->
   <link name="front_right_wheel">
@@ -126,8 +117,4 @@
     <axis xyz="0 1 0"/>
   </joint>
-  <!-- Gazebo 材质 - 左后轮 -->
-  <gazebo reference="rear_left_wheel">
-    <material>Gazebo/Black</material>
-  </gazebo>
   <!-- 左后轮 -->
   <link name="rear_left_wheel">
@@ -163,8 +150,4 @@
     <axis xyz="0 1 0"/>
   </joint>
-  <!-- Gazebo 材质 - 右后轮 -->
-  <gazebo reference="rear_right_wheel">
-    <material>Gazebo/Black</material>
-  </gazebo>
   <!-- 右后轮 -->
   <link name="rear_right_wheel">
@@ -200,5 +183,3 @@
     <axis xyz="0 1 0"/>
   </joint>
-  <xacro:include filename="$(find robot_description)/urdf/robot.ros2_control.xacro" />
-  <xacro:robot_ros2_control />
 </robot>
