Commit message: 修复深度摄像头显示问题

File: src/robot_description/urdf/model/robot.camera.xacro (robot description, xacro)
@@ -80,6 +80,5 @@
     <parent link="camera_link"/>
     <child link="camera_optical_link"/>
-    <!-- ROS 光学坐标系 - x向前, y向左, z向上 (绕 Y 轴旋转 -90°) -->
-    <origin xyz="0 0 0" rpy="0 -1.570795 0"/>
+    <origin xyz="0 0 0" rpy="-1.570795 0 -1.570795"/>
   </joint>
   <!-- ========== Gazebo 材质 ========== -->

Commit message: 添加了深度摄像头避障(待完善)

File: src/robot_description/urdf/model/robot.camera.xacro (robot description, xacro)
@@ -69,9 +69,9 @@
     </inertial>
   </link>
-  <!-- 相机与支架的固定关节 -->
+  <!-- 相机与支架的固定关节 (向下倾斜15度检测低矮障碍物) -->
   <joint name="camera_joint" type="fixed">
     <parent link="camera_bracket"/>
     <child link="camera_link"/>
-    <origin xyz="0 0 ${camera_bracket_height/2 + camera_box_size/2}" rpy="0 0 0"/>
+    <origin xyz="0 0 ${camera_bracket_height/2 + camera_box_size/2}" rpy="0 -0.26 0"/>
   </joint>
   <!-- ========== 相机光学坐标框架 (ROS 相机惯例) ========== -->

File: src/robot_description/urdf/plugin/robot.camera.gazebo.xacro (robot description, xacro)
@@ -4,25 +4,31 @@
     <gazebo reference="camera_link">
       <sensor type="depth" name="camera_sensor">
-        <plugin name="depth_camera" filename="libgazebo_ros_camera.so">
-          <frame_name>camera_optical_link</frame_name>
-        </plugin>
-        <always_on>true</always_on>
         <update_rate>10</update_rate>
-        <camera name="camera">
+        <camera>
           <horizontal_fov>1.5009831567</horizontal_fov>
           <image>
             <width>800</width>
             <height>600</height>
-            <format>R8G8B8</format>
           </image>
-          <distortion>
-            <k1>0.0</k1>
-            <k2>0.0</k2>
-            <k3>0.0</k3>
-            <p1>0.0</p1>
-            <p2>0.0</p2>
-            <center>0.5 0.5</center>
-          </distortion>
+          <clip>
+            <near>0.05</near>
+            <far>8.0</far>
+          </clip>
         </camera>
+        <plugin name="depth_camera" filename="libgazebo_ros_camera.so">
+          <ros>
+            <namespace>/camera</namespace>
+            <remapping>image_raw:=image_raw</remapping>
+            <remapping>depth/image_raw:=depth/image_raw</remapping>
+            <remapping>depth/points:=depth/points</remapping>
+            <remapping>camera_info:=camera_info</remapping>
+            <remapping>depth/camera_info:=depth/camera_info</remapping>
+          </ros>
+          <camera_name>camera</camera_name>
+          <frame_name>camera_optical_link</frame_name>
+          <hack_baseline>0.07</hack_baseline>
+          <min_depth>0.001</min_depth>
+          <max_depth>8.0</max_depth>
+        </plugin>
       </sensor>
     </gazebo>

Commit message: 修复了深度避障的一些问题

File: src/robot_description/urdf/model/robot.camera.xacro (robot description, xacro)
@@ -69,9 +69,9 @@
     </inertial>
   </link>
-  <!-- 相机与支架的固定关节 (向下倾斜15度检测低矮障碍物) -->
+  <!-- 相机与支架的固定关节-->
   <joint name="camera_joint" type="fixed">
     <parent link="camera_bracket"/>
     <child link="camera_link"/>
-    <origin xyz="0 0 ${camera_bracket_height/2 + camera_box_size/2}" rpy="0 -0.26 0"/>
+    <origin xyz="0 0 ${camera_bracket_height/2 + camera_box_size/2}" rpy="0 0 0"/>
   </joint>
   <!-- ========== 相机光学坐标框架 (ROS 相机惯例) ========== -->

File: src/robot_description/urdf/model/robot.lidar.xacro (robot description, xacro)
@@ -8,5 +8,5 @@
   <!-- ========== 支架属性 ========== -->
   <xacro:property name="bracket_radius" value="0.015"/>
-  <xacro:property name="bracket_height" value="0.060"/>
+  <xacro:property name="bracket_height" value="0.35"/>
   <xacro:property name="bracket_mass" value="0.02"/>
   <!-- ========== 支架链接 ========== -->
