Commit message: 优化了模型

File: src/robot_description/urdf/model/robot.lidar.xacro (robot description, xacro)
@@ -41,5 +41,5 @@
     <parent link="base_link"/>
     <child link="lidar_bracket"/>
-    <origin xyz="0 0 ${chassis_height/2 + bracket_height/2}" rpy="0 0 0"/>
+    <origin xyz="${-(chassis_length/2 - 0.05)} 0 ${chassis_height/2 + bracket_height/2}" rpy="0 0 0"/>
   </joint>
   <!-- ========== 激光雷达传感器链接 ========== -->

File: src/robot_description/urdf/model/robot.model.xacro (robot description, xacro)
@@ -24,4 +24,14 @@
   <!-- ========== 机械臂 ========== -->
   <xacro:include filename="robot.arm.xacro"/>
+  <!-- ========== 侧边桶子 ========== -->
+  <xacro:include filename="robot.barrel.xacro"/>
+  <xacro:barrel name="left_barrel" y_sign="1"/>
+  <xacro:barrel name="right_barrel" y_sign="-1"/>
+  <gazebo reference="left_barrel">
+    <material>Gazebo/DarkGrey</material>
+  </gazebo>
+  <gazebo reference="right_barrel">
+    <material>Gazebo/DarkGrey</material>
+  </gazebo>
   <!-- ========== 深度相机（挂在机械臂末端 arm_link3 上） ========== -->
   <xacro:include filename="robot.camera.xacro"/>
