Commit message: 将深度摄像头安装至机械臂上

File: src/robot_description/urdf/model/robot.arm.xacro (robot description, xacro)
@@ -53,4 +53,7 @@
   </joint>
   <xacro:arm_link name="arm_link0" length="${arm_l1}" mass="${arm_m0}" color="0.1 0.1 0.1"/>
+  <gazebo reference="arm_link0">
+    <material>Gazebo/DarkGrey</material>
+  </gazebo>
   <joint name="arm_shoulder_joint" type="revolute">
     <parent link="arm_link0"/>
@@ -61,4 +64,7 @@
   </joint>
   <xacro:arm_link name="arm_link1" length="${arm_l2}" mass="${arm_m1}" color="0.5 0.5 0.5"/>
+  <gazebo reference="arm_link1">
+    <material>Gazebo/Grey</material>
+  </gazebo>
   <joint name="arm_elbow_joint" type="revolute">
     <parent link="arm_link1"/>
@@ -69,4 +75,7 @@
   </joint>
   <xacro:arm_link name="arm_link2" length="${arm_l3}" mass="${arm_m2}" color="0.1 0.1 0.1"/>
+  <gazebo reference="arm_link2">
+    <material>Gazebo/DarkGrey</material>
+  </gazebo>
   <joint name="arm_wrist_joint" type="revolute">
     <parent link="arm_link2"/>
@@ -77,3 +86,6 @@
   </joint>
   <xacro:arm_link name="arm_link3" length="${arm_l4}" mass="${arm_m3}" color="0.5 0.5 0.5"/>
+  <gazebo reference="arm_link3">
+    <material>Gazebo/Grey</material>
+  </gazebo>
 </robot>

File: src/robot_description/urdf/model/robot.camera.xacro (robot description, xacro)
@@ -36,9 +36,9 @@
     </inertial>
   </link>
-  <!-- 支架与底盘的固定关节 (前方偏移) -->
+  <!-- 支架固定在 arm_link3 面积最大的侧面 (+x 面) -->
   <joint name="camera_bracket_joint" type="fixed">
-    <parent link="base_link"/>
+    <parent link="arm_link3"/>
     <child link="camera_bracket"/>
-    <origin xyz="${chassis_length/2 - camera_bracket_length/2} 0 ${chassis_height/2 + camera_bracket_height/2}" rpy="0 0 0"/>
+    <origin xyz="${-arm_w/2 - camera_bracket_height/2} 0 ${arm_l4/2}" rpy="0 ${-PI/2} 0"/>
   </joint>
   <!-- ========== 相机链接 ========== -->

File: src/robot_description/urdf/model/robot.model.xacro (robot description, xacro)
@@ -22,7 +22,7 @@
   <!-- ========== 激光雷达 ========== -->
   <xacro:include filename="robot.lidar.xacro"/>
-  <!-- ========== 深度相机 ========== -->
-  <xacro:include filename="robot.camera.xacro"/>
   <!-- ========== 机械臂 ========== -->
   <xacro:include filename="robot.arm.xacro"/>
+  <!-- ========== 深度相机（挂在机械臂末端 arm_link3 上） ========== -->
+  <xacro:include filename="robot.camera.xacro"/>
 </robot>

Commit message: 修改了模型

File: src/robot_description/urdf/model/robot.arm.xacro (robot description, xacro)
@@ -5,10 +5,12 @@
   <xacro:property name="arm_l2" value="0.129416"/>
   <xacro:property name="arm_l3" value="0.129444"/>
-  <xacro:property name="arm_l4" value="0.1138648"/>
+  <xacro:property name="arm_l4" value="0.0569324"/>
+  <xacro:property name="arm_l5" value="0.0569324"/>
   <xacro:property name="arm_w" value="0.030"/>
   <xacro:property name="arm_m0" value="0.3"/>
   <xacro:property name="arm_m1" value="0.4"/>
   <xacro:property name="arm_m2" value="0.3"/>
-  <xacro:property name="arm_m3" value="0.2"/>
+  <xacro:property name="arm_m3" value="0.1"/>
+  <xacro:property name="arm_m4" value="0.1"/>
   <xacro:property name="arm_origin_x" value="${chassis_length/2 - 0.05}"/>
   <xacro:property name="arm_origin_y" value="0.0"/>
@@ -89,3 +91,38 @@
     <material>Gazebo/Grey</material>
   </gazebo>
+  <joint name="arm_tool_rotate_joint" type="revolute">
+    <parent link="arm_link3"/>
+    <child link="arm_link4"/>
+    <origin xyz="0 0 ${arm_l4}" rpy="0 0 0"/>
+    <axis xyz="0 0 1"/>
+    <limit lower="${-PI}" upper="${PI}" effort="10" velocity="3.14"/>
+  </joint>
+  <xacro:arm_link name="arm_link4" length="${arm_l5}" mass="${arm_m4}" color="0.5 0.5 0.5"/>
+  <gazebo reference="arm_link4">
+    <material>Gazebo/Grey</material>
+  </gazebo>
+  <joint name="virtual_tool_roll_joint" type="revolute">
+    <parent link="arm_link4"/>
+    <child link="tool_roll_link"/>
+    <origin xyz="0 0 ${arm_l5}" rpy="0 0 0"/>
+    <axis xyz="1 0 0"/>
+    <limit lower="${-PI}" upper="${PI}" effort="1" velocity="3.14"/>
+  </joint>
+  <link name="tool_roll_link"/>
+  <joint name="virtual_tool_pitch_joint" type="revolute">
+    <parent link="tool_roll_link"/>
+    <child link="tool_pitch_link"/>
+    <origin xyz="0 0 0" rpy="0 0 0"/>
+    <axis xyz="0 1 0"/>
+    <limit lower="${-PI}" upper="${PI}" effort="1" velocity="3.14"/>
+  </joint>
+  <link name="tool_pitch_link"/>
+  <joint name="virtual_tool_yaw_joint" type="revolute">
+    <parent link="tool_pitch_link"/>
+    <child link="tool0"/>
+    <origin xyz="0 0 0" rpy="0 0 0"/>
+    <axis xyz="0 0 1"/>
+    <limit lower="${-PI}" upper="${PI}" effort="1" velocity="3.14"/>
+  </joint>
+  <link name="tool0"/>
 </robot>

File: src/robot_description/urdf/model/robot.camera.xacro (robot description, xacro)
@@ -36,9 +36,9 @@
     </inertial>
   </link>
-  <!-- 支架固定在 arm_link3 面积最大的侧面 (+x 面) -->
+  <!-- 支架固定在 arm_link4 基部侧面 -->
   <joint name="camera_bracket_joint" type="fixed">
-    <parent link="arm_link3"/>
+    <parent link="arm_link4"/>
     <child link="camera_bracket"/>
-    <origin xyz="${-arm_w/2 - camera_bracket_height/2} 0 ${arm_l4/2}" rpy="0 ${-PI/2} 0"/>
+    <origin xyz="${-arm_w/2 - camera_bracket_height/2} 0 0" rpy="0 ${-PI/2} 0"/>
   </joint>
   <!-- ========== 相机链接 ========== -->

File: src/robot_description/urdf/model/robot.model.xacro (robot description, xacro)
@@ -34,5 +34,5 @@
     <material>Gazebo/DarkGrey</material>
   </gazebo>
-  <!-- ========== 深度相机（挂在机械臂末端 arm_link3 上） ========== -->
+  <!-- ========== 深度相机（挂在机械臂末端 arm_link4 上） ========== -->
   <xacro:include filename="robot.camera.xacro"/>
 </robot>

File: src/robot_moveit_config/config/robot_arm_moveit.ros2_control.xacro (robot description, xacro)
@@ -50,18 +50,4 @@
                 <state_interface name="velocity"/>
             </joint>
-            <joint name="virtual_tool_pitch_joint">
-                <command_interface name="position"/>
-                <state_interface name="position">
-                  <param name="initial_value">${initial_positions['virtual_tool_pitch_joint']}</param>
-                </state_interface>
-                <state_interface name="velocity"/>
-            </joint>
-            <joint name="virtual_tool_yaw_joint">
-                <command_interface name="position"/>
-                <state_interface name="position">
-                  <param name="initial_value">${initial_positions['virtual_tool_yaw_joint']}</param>
-                </state_interface>
-                <state_interface name="velocity"/>
-            </joint>
         </ros2_control>
     </xacro:macro>

Commit message: 修改机械臂模型

File: src/robot_description/urdf/model/robot.arm.xacro (robot description, xacro)
@@ -8,4 +8,11 @@
   <xacro:property name="arm_l5" value="0.0569324"/>
   <xacro:property name="arm_w" value="0.030"/>
+  <xacro:property name="gripper_base_length" value="${arm_w}"/>
+  <xacro:property name="gripper_base_width" value="0.070"/>
+  <xacro:property name="gripper_base_height" value="0.018"/>
+  <xacro:property name="gripper_finger_length" value="${arm_l5 - gripper_base_height}"/>
+  <xacro:property name="gripper_finger_width" value="${arm_w}"/>
+  <xacro:property name="gripper_finger_thickness" value="0.010"/>
+  <xacro:property name="gripper_finger_y_offset" value="0.026"/>
   <xacro:property name="arm_m0" value="0.3"/>
   <xacro:property name="arm_m1" value="0.4"/>
@@ -13,4 +20,6 @@
   <xacro:property name="arm_m3" value="0.1"/>
   <xacro:property name="arm_m4" value="0.1"/>
+  <xacro:property name="gripper_base_mass" value="${arm_m4 * 0.70}"/>
+  <xacro:property name="gripper_finger_mass" value="${arm_m4 * 0.15}"/>
   <xacro:property name="arm_origin_x" value="${chassis_length/2 - 0.05}"/>
   <xacro:property name="arm_origin_y" value="0.0"/>
@@ -22,4 +31,9 @@
              izz="${mass/6.0 * w*w}"/>
   </xacro:macro>
+  <xacro:macro name="box_inertia_xyz" params="mass x y z">
+    <inertia ixx="${mass/12.0 * (y*y + z*z)}" ixy="0" ixz="0"
+             iyy="${mass/12.0 * (x*x + z*z)}" iyz="0"
+             izz="${mass/12.0 * (x*x + y*y)}"/>
+  </xacro:macro>
   <!-- ========== 连杆宏 ========== -->
   <xacro:macro name="arm_link" params="name length mass color">
@@ -47,4 +61,33 @@
     </link>
   </xacro:macro>
+  <xacro:macro name="gripper_finger" params="name y_sign">
+    <joint name="${name}_joint" type="fixed">
+      <parent link="arm_link4"/>
+      <child link="${name}"/>
+      <origin xyz="0 ${y_sign * gripper_finger_y_offset} ${gripper_base_height}" rpy="0 0 0"/>
+    </joint>
+    <link name="${name}">
+      <visual>
+        <origin xyz="0 0 ${gripper_finger_length/2}" rpy="0 0 0"/>
+        <geometry>
+          <box size="${gripper_finger_width} ${gripper_finger_thickness} ${gripper_finger_length}"/>
+        </geometry>
+        <material name="gripper_finger_black">
+          <color rgba="0.05 0.05 0.05 1.0"/>
+        </material>
+      </visual>
+      <collision>
+        <origin xyz="0 0 ${gripper_finger_length/2}" rpy="0 0 0"/>
+        <geometry>
+          <box size="${gripper_finger_width} ${gripper_finger_thickness} ${gripper_finger_length}"/>
+        </geometry>
+      </collision>
+      <inertial>
+        <origin xyz="0 0 ${gripper_finger_length/2}" rpy="0 0 0"/>
+        <mass value="${gripper_finger_mass}"/>
+        <xacro:box_inertia_xyz mass="${gripper_finger_mass}" x="${gripper_finger_width}" y="${gripper_finger_thickness}" z="${gripper_finger_length}"/>
+      </inertial>
+    </link>
+  </xacro:macro>
   <joint name="arm_base_joint" type="revolute">
     <parent link="base_link"/>
@@ -98,7 +141,36 @@
     <limit lower="${-PI}" upper="${PI}" effort="10" velocity="3.14"/>
   </joint>
-  <xacro:arm_link name="arm_link4" length="${arm_l5}" mass="${arm_m4}" color="0.5 0.5 0.5"/>
+  <link name="arm_link4">
+    <visual>
+      <origin xyz="0 0 ${gripper_base_height/2}" rpy="0 0 0"/>
+      <geometry>
+        <box size="${gripper_base_length} ${gripper_base_width} ${gripper_base_height}"/>
+      </geometry>
+      <material name="gripper_base_grey">
+        <color rgba="0.45 0.45 0.45 1.0"/>
+      </material>
+    </visual>
+    <collision>
+      <origin xyz="0 0 ${gripper_base_height/2}" rpy="0 0 0"/>
+      <geometry>
+        <box size="${gripper_base_length} ${gripper_base_width} ${gripper_base_height}"/>
+      </geometry>
+    </collision>
+    <inertial>
+      <origin xyz="0 0 ${gripper_base_height/2}" rpy="0 0 0"/>
+      <mass value="${gripper_base_mass}"/>
+      <xacro:box_inertia_xyz mass="${gripper_base_mass}" x="${gripper_base_length}" y="${gripper_base_width}" z="${gripper_base_height}"/>
+    </inertial>
+  </link>
   <gazebo reference="arm_link4">
     <material>Gazebo/Grey</material>
+  </gazebo>
+  <xacro:gripper_finger name="left_gripper_finger" y_sign="1"/>
+  <xacro:gripper_finger name="right_gripper_finger" y_sign="-1"/>
+  <gazebo reference="left_gripper_finger">
+    <material>Gazebo/Black</material>
+  </gazebo>
+  <gazebo reference="right_gripper_finger">
+    <material>Gazebo/Black</material>
   </gazebo>
   <joint name="virtual_tool_roll_joint" type="revolute">

File: src/robot_description/urdf/model/robot.camera.xacro (robot description, xacro)
@@ -40,5 +40,5 @@
     <parent link="arm_link4"/>
     <child link="camera_bracket"/>
-    <origin xyz="${-arm_w/2 - camera_bracket_height/2} 0 0" rpy="0 ${-PI/2} 0"/>
+    <origin xyz="${-gripper_base_length/2 - camera_bracket_height/2} 0 0" rpy="0 ${-PI/2} 0"/>
   </joint>
   <!-- ========== 相机链接 ========== -->

File: src/robot_description/urdf/robot_arm_moveit.urdf (robot description, URDF)
Before this commit: robot robot_arm_moveit, 12 links, 11 joints
Links:
- added link left_gripper_finger, mass 0.015; collision box size=0.03 0.01 0.0389324; visual box size=0.03 0.01 0.0389324
- added link right_gripper_finger, mass 0.015; collision box size=0.03 0.01 0.0389324; visual box size=0.03 0.01 0.0389324
- link arm_link4: mass 0.1 -> 0.07; geometry collision box size=0.03 0.07 0.018; visual box size=0.03 0.07 0.018
Joints:
- added joint left_gripper_finger_joint: type fixed, parent arm_link4, child left_gripper_finger, origin xyz=0 0.026 0.018 rpy=0 0 0
- added joint right_gripper_finger_joint: type fixed, parent arm_link4, child right_gripper_finger, origin xyz=0 -0.026 0.018 rpy=0 0 0

Commit message: 去除了自己写的ik

File: src/robot_description/urdf/model/robot.arm.xacro (robot description, xacro)
@@ -91,10 +91,10 @@
     </link>
   </xacro:macro>
-  <joint name="arm_base_joint" type="revolute">
+  <joint name="arm_base_joint" type="continuous">
     <parent link="base_link"/>
     <child link="arm_link0"/>
     <origin xyz="${arm_origin_x} ${arm_origin_y} ${arm_origin_z}" rpy="0 0 0"/>
     <axis xyz="0 0 1"/>
-    <limit lower="${-PI}" upper="${PI}" effort="10" velocity="3.14"/>
+    <limit effort="10" velocity="3.14"/>
   </joint>
   <xacro:arm_link name="arm_link0" length="${arm_l1}" mass="${arm_m0}" color="0.1 0.1 0.1"/>
@@ -102,10 +102,10 @@
     <material>Gazebo/DarkGrey</material>
   </gazebo>
-  <joint name="arm_shoulder_joint" type="revolute">
+  <joint name="arm_shoulder_joint" type="continuous">
     <parent link="arm_link0"/>
     <child link="arm_link1"/>
     <origin xyz="0 0 ${arm_l1}" rpy="0 0 0"/>
     <axis xyz="0 1 0"/>
-    <limit lower="${-PI/2}" upper="${PI}" effort="10" velocity="3.14"/>
+    <limit effort="10" velocity="3.14"/>
   </joint>
   <xacro:arm_link name="arm_link1" length="${arm_l2}" mass="${arm_m1}" color="0.5 0.5 0.5"/>
@@ -113,10 +113,10 @@
     <material>Gazebo/Grey</material>
   </gazebo>
-  <joint name="arm_elbow_joint" type="revolute">
+  <joint name="arm_elbow_joint" type="continuous">
     <parent link="arm_link1"/>
     <child link="arm_link2"/>
     <origin xyz="0 0 ${arm_l2}" rpy="0 0 0"/>
     <axis xyz="0 1 0"/>
-    <limit lower="0" upper="${PI}" effort="10" velocity="3.14"/>
+    <limit effort="10" velocity="3.14"/>
   </joint>
   <xacro:arm_link name="arm_link2" length="${arm_l3}" mass="${arm_m2}" color="0.1 0.1 0.1"/>
@@ -124,10 +124,10 @@
     <material>Gazebo/DarkGrey</material>
   </gazebo>
-  <joint name="arm_wrist_joint" type="revolute">
+  <joint name="arm_wrist_joint" type="continuous">
     <parent link="arm_link2"/>
     <child link="arm_link3"/>
     <origin xyz="0 0 ${arm_l3}" rpy="0 0 0"/>
     <axis xyz="0 1 0"/>
-    <limit lower="0" upper="${PI}" effort="10" velocity="3.14"/>
+    <limit effort="10" velocity="3.14"/>
   </joint>
   <xacro:arm_link name="arm_link3" length="${arm_l4}" mass="${arm_m3}" color="0.5 0.5 0.5"/>
@@ -135,10 +135,10 @@
     <material>Gazebo/Grey</material>
   </gazebo>
-  <joint name="arm_tool_rotate_joint" type="revolute">
+  <joint name="arm_tool_rotate_joint" type="continuous">
     <parent link="arm_link3"/>
     <child link="arm_link4"/>
     <origin xyz="0 0 ${arm_l4}" rpy="0 0 0"/>
     <axis xyz="0 0 1"/>
-    <limit lower="${-PI}" upper="${PI}" effort="10" velocity="3.14"/>
+    <limit effort="10" velocity="3.14"/>
   </joint>
   <link name="arm_link4">
@@ -175,10 +175,10 @@
     <material>Gazebo/Black</material>
   </gazebo>
-  <joint name="virtual_tool_roll_joint" type="revolute">
+  <joint name="virtual_tool_roll_joint" type="continuous">
     <parent link="arm_link4"/>
     <child link="tool_roll_link"/>
     <origin xyz="0 0 ${arm_l5}" rpy="0 0 0"/>
     <axis xyz="1 0 0"/>
-    <limit lower="${-PI}" upper="${PI}" effort="1" velocity="3.14"/>
+    <limit effort="1" velocity="3.14"/>
   </joint>
   <link name="tool_roll_link">
@@ -188,10 +188,10 @@
     </inertial>
   </link>
-  <joint name="virtual_tool_pitch_joint" type="revolute">
+  <joint name="virtual_tool_pitch_joint" type="continuous">
     <parent link="tool_roll_link"/>
     <child link="tool_pitch_link"/>
     <origin xyz="0 0 0" rpy="0 0 0"/>
     <axis xyz="0 1 0"/>
-    <limit lower="${-PI}" upper="${PI}" effort="1" velocity="3.14"/>
+    <limit effort="1" velocity="3.14"/>
   </joint>
   <link name="tool_pitch_link">
@@ -201,10 +201,10 @@
     </inertial>
   </link>
-  <joint name="virtual_tool_yaw_joint" type="revolute">
+  <joint name="virtual_tool_yaw_joint" type="continuous">
     <parent link="tool_pitch_link"/>
     <child link="tool0"/>
     <origin xyz="0 0 0" rpy="0 0 0"/>
     <axis xyz="0 0 1"/>
-    <limit lower="${-PI}" upper="${PI}" effort="1" velocity="3.14"/>
+    <limit effort="1" velocity="3.14"/>
   </joint>
   <link name="tool0">

Commit message: 修复bug

File: src/robot_description/urdf/model/robot.arm.xacro (robot description, xacro)
@@ -23,4 +23,6 @@
   <xacro:property name="gripper_finger_mass" value="${arm_m4 * 0.15}"/>
   <xacro:property name="tool_virtual_mass" value="0.001"/>
+  <xacro:property name="tool_virtual_joint_damping" value="5.0"/>
+  <xacro:property name="tool_virtual_joint_friction" value="0.1"/>
   <xacro:property name="arm_origin_x" value="${chassis_length/2 - 0.05}"/>
   <xacro:property name="arm_origin_y" value="0.0"/>
@@ -181,4 +183,5 @@
     <axis xyz="1 0 0"/>
     <limit effort="1" velocity="3.14"/>
+    <dynamics damping="${tool_virtual_joint_damping}" friction="${tool_virtual_joint_friction}"/>
   </joint>
   <link name="tool_roll_link">
@@ -194,4 +197,5 @@
     <axis xyz="0 1 0"/>
     <limit effort="1" velocity="3.14"/>
+    <dynamics damping="${tool_virtual_joint_damping}" friction="${tool_virtual_joint_friction}"/>
   </joint>
   <link name="tool_pitch_link">
@@ -207,4 +211,5 @@
     <axis xyz="0 0 1"/>
     <limit effort="1" velocity="3.14"/>
+    <dynamics damping="${tool_virtual_joint_damping}" friction="${tool_virtual_joint_friction}"/>
   </joint>
   <link name="tool0">

Commit message: 修复机械臂控制bug

File: src/robot_description/urdf/model/robot.arm.xacro (robot description, xacro)
@@ -93,10 +93,10 @@
     </link>
   </xacro:macro>
-  <joint name="arm_base_joint" type="continuous">
+  <joint name="arm_base_joint" type="revolute">
     <parent link="base_link"/>
     <child link="arm_link0"/>
     <origin xyz="${arm_origin_x} ${arm_origin_y} ${arm_origin_z}" rpy="0 0 0"/>
     <axis xyz="0 0 1"/>
-    <limit effort="10" velocity="3.14"/>
+    <limit lower="-3.141592653589793" upper="3.141592653589793" effort="10" velocity="3.14"/>
   </joint>
   <xacro:arm_link name="arm_link0" length="${arm_l1}" mass="${arm_m0}" color="0.1 0.1 0.1"/>
@@ -104,10 +104,10 @@
     <material>Gazebo/DarkGrey</material>
   </gazebo>
-  <joint name="arm_shoulder_joint" type="continuous">
+  <joint name="arm_shoulder_joint" type="revolute">
     <parent link="arm_link0"/>
     <child link="arm_link1"/>
     <origin xyz="0 0 ${arm_l1}" rpy="0 0 0"/>
     <axis xyz="0 1 0"/>
-    <limit effort="10" velocity="3.14"/>
+    <limit lower="-2.0943951023931953" upper="2.0943951023931953" effort="10" velocity="3.14"/>
   </joint>
   <xacro:arm_link name="arm_link1" length="${arm_l2}" mass="${arm_m1}" color="0.5 0.5 0.5"/>
@@ -115,10 +115,10 @@
     <material>Gazebo/Grey</material>
   </gazebo>
-  <joint name="arm_elbow_joint" type="continuous">
+  <joint name="arm_elbow_joint" type="revolute">
     <parent link="arm_link1"/>
     <child link="arm_link2"/>
     <origin xyz="0 0 ${arm_l2}" rpy="0 0 0"/>
     <axis xyz="0 1 0"/>
-    <limit effort="10" velocity="3.14"/>
+    <limit lower="-2.0943951023931953" upper="2.0943951023931953" effort="10" velocity="3.14"/>
   </joint>
   <xacro:arm_link name="arm_link2" length="${arm_l3}" mass="${arm_m2}" color="0.1 0.1 0.1"/>
@@ -126,10 +126,10 @@
     <material>Gazebo/DarkGrey</material>
   </gazebo>
-  <joint name="arm_wrist_joint" type="continuous">
+  <joint name="arm_wrist_joint" type="revolute">
     <parent link="arm_link2"/>
     <child link="arm_link3"/>
     <origin xyz="0 0 ${arm_l3}" rpy="0 0 0"/>
     <axis xyz="0 1 0"/>
-    <limit effort="10" velocity="3.14"/>
+    <limit lower="-2.0943951023931953" upper="2.0943951023931953" effort="10" velocity="3.14"/>
   </joint>
   <xacro:arm_link name="arm_link3" length="${arm_l4}" mass="${arm_m3}" color="0.5 0.5 0.5"/>
@@ -137,10 +137,10 @@
     <material>Gazebo/Grey</material>
   </gazebo>
-  <joint name="arm_tool_rotate_joint" type="continuous">
+  <joint name="arm_tool_rotate_joint" type="revolute">
     <parent link="arm_link3"/>
     <child link="arm_link4"/>
     <origin xyz="0 0 ${arm_l4}" rpy="0 0 0"/>
     <axis xyz="0 0 1"/>
-    <limit effort="10" velocity="3.14"/>
+    <limit lower="-2.0943951023931953" upper="2.0943951023931953" effort="10" velocity="3.14"/>
   </joint>
   <link name="arm_link4">
