Commit message: 添加了ekf

File: src/robot_description/urdf/model/robot.chassis.xacro (robot description, xacro)
@@ -35,4 +35,10 @@
     <origin xyz="0.0 0.0 ${wheel_z_offset + wheel_radius - 0.001}" rpy="0 0 0" />
   </joint>
+  <link name="imu_link" />
+  <joint name="imu_joint" type="fixed">
+    <parent link="base_link" />
+    <child link="imu_link" />
+    <origin xyz="0 0 0" rpy="0 0 0" />
+  </joint>
   <!-- ========== Gazebo 材质 ========== -->
   <gazebo reference="base_link">
