Commit message: moveit接入gazebo

File: src/robot_description/urdf/control/arm.joints.xacro (robot description, xacro)
@@ -22,4 +22,24 @@
             <state_interface name="velocity"/>
         </joint>
+        <joint name="arm_tool_rotate_joint">
+            <command_interface name="position"/>
+            <state_interface name="position"/>
+            <state_interface name="velocity"/>
+        </joint>
+        <joint name="virtual_tool_roll_joint">
+            <command_interface name="position"/>
+            <state_interface name="position"/>
+            <state_interface name="velocity"/>
+        </joint>
+        <joint name="virtual_tool_pitch_joint">
+            <command_interface name="position"/>
+            <state_interface name="position"/>
+            <state_interface name="velocity"/>
+        </joint>
+        <joint name="virtual_tool_yaw_joint">
+            <command_interface name="position"/>
+            <state_interface name="position"/>
+            <state_interface name="velocity"/>
+        </joint>
     </xacro:macro>
 </robot>

File: src/robot_description/urdf/control/gazebo.control.xacro (robot description, xacro)
@@ -34,4 +34,5 @@
     <!-- ===== 机械臂 ros2_control 接口 ===== -->
     <xacro:include filename="arm.joints.xacro"/>
+    <xacro:include filename="wheel.joints.xacro"/>
     <!-- ===== 机械臂：gazebo_ros2_control ===== -->
     <!-- ros2_control 放在 robot 级别，plugin 内部只放 parameters -->
@@ -42,4 +43,5 @@
             </hardware>
             <xacro:arm_joints/>
+            <xacro:wheel_state_joints/>
         </ros2_control>
         <gazebo>

File: src/robot_description/urdf/control/wheel.joints.xacro (robot description, xacro)
@@ -28,3 +28,21 @@
         </joint>
     </xacro:macro>
+    <xacro:macro name="wheel_state_joints">
+        <joint name="front_left_wheel_joint">
+            <state_interface name="position"/>
+            <state_interface name="velocity"/>
+        </joint>
+        <joint name="front_right_wheel_joint">
+            <state_interface name="position"/>
+            <state_interface name="velocity"/>
+        </joint>
+        <joint name="rear_left_wheel_joint">
+            <state_interface name="position"/>
+            <state_interface name="velocity"/>
+        </joint>
+        <joint name="rear_right_wheel_joint">
+            <state_interface name="position"/>
+            <state_interface name="velocity"/>
+        </joint>
+    </xacro:macro>
 </robot>

File: src/robot_description/urdf/model/robot.arm.xacro (robot description, xacro)
@@ -22,4 +22,5 @@
   <xacro:property name="gripper_base_mass" value="${arm_m4 * 0.70}"/>
   <xacro:property name="gripper_finger_mass" value="${arm_m4 * 0.15}"/>
+  <xacro:property name="tool_virtual_mass" value="0.001"/>
   <xacro:property name="arm_origin_x" value="${chassis_length/2 - 0.05}"/>
   <xacro:property name="arm_origin_y" value="0.0"/>
@@ -181,5 +182,10 @@
     <limit lower="${-PI}" upper="${PI}" effort="1" velocity="3.14"/>
   </joint>
-  <link name="tool_roll_link"/>
+  <link name="tool_roll_link">
+    <inertial>
+      <mass value="${tool_virtual_mass}"/>
+      <inertia ixx="1e-6" ixy="0" ixz="0" iyy="1e-6" iyz="0" izz="1e-6"/>
+    </inertial>
+  </link>
   <joint name="virtual_tool_pitch_joint" type="revolute">
     <parent link="tool_roll_link"/>
@@ -189,5 +195,10 @@
     <limit lower="${-PI}" upper="${PI}" effort="1" velocity="3.14"/>
   </joint>
-  <link name="tool_pitch_link"/>
+  <link name="tool_pitch_link">
+    <inertial>
+      <mass value="${tool_virtual_mass}"/>
+      <inertia ixx="1e-6" ixy="0" ixz="0" iyy="1e-6" iyz="0" izz="1e-6"/>
+    </inertial>
+  </link>
   <joint name="virtual_tool_yaw_joint" type="revolute">
     <parent link="tool_pitch_link"/>
@@ -197,4 +208,9 @@
     <limit lower="${-PI}" upper="${PI}" effort="1" velocity="3.14"/>
   </joint>
-  <link name="tool0"/>
+  <link name="tool0">
+    <inertial>
+      <mass value="${tool_virtual_mass}"/>
+      <inertia ixx="1e-6" ixy="0" ixz="0" iyy="1e-6" iyz="0" izz="1e-6"/>
+    </inertial>
+  </link>
 </robot>

Commit message: 一点小优化

File: src/robot_description/urdf/control/arm.joints.xacro (robot description, xacro)
@@ -1,43 +1,60 @@
 <?xml version="1.0"?>
 <robot xmlns:xacro="http://www.ros.org/wiki/xacro">
-    <xacro:macro name="arm_joints">
+    <xacro:macro name="arm_joints" params="initial_positions_file">
+        <xacro:property name="initial_positions" value="${xacro.load_yaml(initial_positions_file)['initial_positions']}"/>
         <joint name="arm_base_joint">
             <command_interface name="position"/>
-            <state_interface name="position"/>
+            <state_interface name="position">
+                <param name="initial_value">${initial_positions['arm_base_joint']}</param>
+            </state_interface>
             <state_interface name="velocity"/>
         </joint>
         <joint name="arm_shoulder_joint">
             <command_interface name="position"/>
-            <state_interface name="position"/>
+            <state_interface name="position">
+                <param name="initial_value">${initial_positions['arm_shoulder_joint']}</param>
+            </state_interface>
             <state_interface name="velocity"/>
         </joint>
         <joint name="arm_elbow_joint">
             <command_interface name="position"/>
-            <state_interface name="position"/>
+            <state_interface name="position">
+                <param name="initial_value">${initial_positions['arm_elbow_joint']}</param>
+            </state_interface>
             <state_interface name="velocity"/>
         </joint>
         <joint name="arm_wrist_joint">
             <command_interface name="position"/>
-            <state_interface name="position"/>
+            <state_interface name="position">
+                <param name="initial_value">${initial_positions['arm_wrist_joint']}</param>
+            </state_interface>
             <state_interface name="velocity"/>
         </joint>
         <joint name="arm_tool_rotate_joint">
             <command_interface name="position"/>
-            <state_interface name="position"/>
+            <state_interface name="position">
+                <param name="initial_value">${initial_positions['arm_tool_rotate_joint']}</param>
+            </state_interface>
             <state_interface name="velocity"/>
         </joint>
         <joint name="virtual_tool_roll_joint">
             <command_interface name="position"/>
-            <state_interface name="position"/>
+            <state_interface name="position">
+                <param name="initial_value">${initial_positions['virtual_tool_roll_joint']}</param>
+            </state_interface>
             <state_interface name="velocity"/>
         </joint>
         <joint name="virtual_tool_pitch_joint">
             <command_interface name="position"/>
-            <state_interface name="position"/>
+            <state_interface name="position">
+                <param name="initial_value">${initial_positions['virtual_tool_pitch_joint']}</param>
+            </state_interface>
             <state_interface name="velocity"/>
         </joint>
         <joint name="virtual_tool_yaw_joint">
             <command_interface name="position"/>
-            <state_interface name="position"/>
+            <state_interface name="position">
+                <param name="initial_value">${initial_positions['virtual_tool_yaw_joint']}</param>
+            </state_interface>
             <state_interface name="velocity"/>
         </joint>

File: src/robot_description/urdf/control/gazebo.control.xacro (robot description, xacro)
@@ -37,10 +37,10 @@
     <!-- ===== 机械臂：gazebo_ros2_control ===== -->
     <!-- ros2_control 放在 robot 级别，plugin 内部只放 parameters -->
-    <xacro:macro name="robot_arm_control">
+    <xacro:macro name="robot_arm_control" params="initial_positions_file">
         <ros2_control name="RobotArmGazeboSystem" type="system">
             <hardware>
                 <plugin>gazebo_ros2_control/GazeboSystem</plugin>
             </hardware>
-            <xacro:arm_joints/>
+            <xacro:arm_joints initial_positions_file="${initial_positions_file}"/>
             <xacro:wheel_state_joints/>
         </ros2_control>

File: src/robot_description/urdf/robot.gazebo.xacro (robot description, xacro)
@@ -1,9 +1,10 @@
 <?xml version="1.0"?>
 <robot name="four_wheel_robot" xmlns:xacro="http://www.ros.org/wiki/xacro">
+  <xacro:arg name="arm_initial_positions_file" default="$(find robot_description)/config/arm_initial_positions.yaml" />
   <!-- 共享模型定义 -->
   <xacro:include filename="$(find robot_description)/urdf/model/robot.model.xacro" />
   <xacro:include filename="$(find robot_description)/urdf/control/gazebo.control.xacro" />
   <xacro:robot_ros2_control />
-  <xacro:robot_arm_control />
+  <xacro:robot_arm_control initial_positions_file="$(arg arm_initial_positions_file)" />
   <!-- 激光雷达 Gazebo 插件 -->
   <xacro:include filename="$(find robot_description)/urdf/plugin/robot.lidar.gazebo.xacro" />
