Commit message: 规范代码

File: src/robot_description/urdf/control/gazebo.control.xacro (robot description, xacro)
@@ -11,5 +11,5 @@
         <gazebo>
             <plugin filename="libgazebo_ros2_control.so" name="gazebo_ros2_control">
-                <parameters>$(find robot_description)/config/gazebo_ros2_controller.yaml</parameters>
+                <parameters>$(find robot_description)/config/robot_gazebo_controllers.yaml</parameters>
                 <ros>
                     <remapping>/robot_diff_drive_controller/cmd_vel_unstamped:=/cmd_vel</remapping>

File: src/robot_description/urdf/robot.model.xacro (robot description, xacro)
@@ -183,3 +183,35 @@
     <axis xyz="0 1 0"/>
   </joint>
+  <!-- ========== Gazebo 材质 ========== -->
+  <gazebo reference="base_link">
+    <material>Gazebo/Grey</material>
+  </gazebo>
+  <gazebo reference="front_left_wheel">
+    <material>Gazebo/Black</material>
+    <mu1 value="20.0"/>
+    <mu2 value="20.0"/>
+    <kp value="1000000000.0"/>
+    <kd value="1.0"/>
+  </gazebo>
+  <gazebo reference="front_right_wheel">
+    <material>Gazebo/Black</material>
+    <mu1 value="20.0"/>
+    <mu2 value="20.0"/>
+    <kp value="1000000000.0"/>
+    <kd value="1.0"/>
+  </gazebo>
+  <gazebo reference="rear_left_wheel">
+    <material>Gazebo/Black</material>
+    <mu1 value="20.0"/>
+    <mu2 value="20.0"/>
+    <kp value="1000000000.0"/>
+    <kd value="1.0"/>
+  </gazebo>
+  <gazebo reference="rear_right_wheel">
+    <material>Gazebo/Black</material>
+    <mu1 value="20.0"/>
+    <mu2 value="20.0"/>
+    <kp value="1000000000.0"/>
+    <kd value="1.0"/>
+  </gazebo>
 </robot>

Commit message: 为gazebo添加机械臂仿真

File: src/robot_description/urdf/control/gazebo.control.xacro (robot description, xacro)
@@ -1,4 +1,5 @@
 <?xml version="1.0"?>
 <robot xmlns:xacro="http://www.ros.org/wiki/xacro">
+    <!-- ===== 底盘：gazebo_ros_diff_drive ===== -->
     <xacro:macro name="robot_ros2_control">
         <gazebo>
@@ -31,3 +32,20 @@
         </gazebo>
     </xacro:macro>
+    <!-- ===== 机械臂 ros2_control 接口 ===== -->
+    <xacro:include filename="arm.joints.xacro"/>
+    <!-- ===== 机械臂：gazebo_ros2_control ===== -->
+    <!-- ros2_control 放在 robot 级别，plugin 内部只放 parameters -->
+    <xacro:macro name="robot_arm_control">
+        <ros2_control name="RobotArmGazeboSystem" type="system">
+            <hardware>
+                <plugin>gazebo_ros2_control/GazeboSystem</plugin>
+            </hardware>
+            <xacro:arm_joints/>
+        </ros2_control>
+        <gazebo>
+            <plugin name="gazebo_ros2_control" filename="libgazebo_ros2_control.so">
+                <parameters>$(find robot_description)/config/robot_gazebo_controllers.yaml</parameters>
+            </plugin>
+        </gazebo>
+    </xacro:macro>
 </robot>

File: src/robot_description/urdf/robot.gazebo.xacro (robot description, xacro)
@@ -3,7 +3,7 @@
   <!-- 共享模型定义 -->
   <xacro:include filename="$(find robot_description)/urdf/model/robot.model.xacro" />
-  <!-- ros2_control hardware interface -->
   <xacro:include filename="$(find robot_description)/urdf/control/gazebo.control.xacro" />
   <xacro:robot_ros2_control />
+  <xacro:robot_arm_control />
   <!-- 激光雷达 Gazebo 插件 -->
   <xacro:include filename="$(find robot_description)/urdf/plugin/robot.lidar.gazebo.xacro" />

Commit message: URDF参照真实机器人

File: src/robot_description/urdf/control/gazebo.control.xacro (robot description, xacro)
@@ -16,6 +16,6 @@
                 <right_joint>rear_right_wheel_joint</right_joint>
                 <!-- kinematics -->
-                <wheel_separation>0.225</wheel_separation>
-                <wheel_separation>0.225</wheel_separation>
+                <wheel_separation>${wheel_y_offset * 2}</wheel_separation>
+                <wheel_separation>${wheel_y_offset * 2}</wheel_separation>
                 <wheel_diameter>${wheel_radius * 2}</wheel_diameter>
                 <wheel_diameter>${wheel_radius * 2}</wheel_diameter>

File: src/robot_description/urdf/model/robot.arm.xacro (robot description, xacro)
@@ -5,10 +5,10 @@
   <xacro:property name="arm_l2" value="0.129416"/>
   <xacro:property name="arm_l3" value="0.129444"/>
-  <xacro:property name="arm_l4" value="0.0569324"/>
-  <xacro:property name="arm_l5" value="0.0569324"/>
+  <xacro:property name="arm_l4" value="0.05448"/>
+  <xacro:property name="arm_l5" value="0.1183848"/>
   <xacro:property name="arm_w" value="0.030"/>
   <xacro:property name="gripper_base_length" value="${arm_w}"/>
   <xacro:property name="gripper_base_width" value="0.070"/>
-  <xacro:property name="gripper_base_height" value="0.018"/>
+  <xacro:property name="gripper_base_height" value="0.0593848"/>
   <xacro:property name="gripper_finger_length" value="${arm_l5 - gripper_base_height}"/>
   <xacro:property name="gripper_finger_width" value="${arm_w}"/>
@@ -25,5 +25,5 @@
   <xacro:property name="tool_virtual_joint_damping" value="5.0"/>
   <xacro:property name="tool_virtual_joint_friction" value="0.1"/>
-  <xacro:property name="arm_origin_x" value="${chassis_length/2 - 0.05}"/>
+  <xacro:property name="arm_origin_x" value="${chassis_length/2 - 0.055}"/>
   <xacro:property name="arm_origin_y" value="0.0"/>
   <xacro:property name="arm_origin_z" value="${chassis_height/2}"/>

File: src/robot_description/urdf/model/robot.barrel.xacro (robot description, xacro)
@@ -2,9 +2,10 @@
 <robot xmlns:xacro="http://www.ros.org/wiki/xacro">
   <!-- ========== 属性 ========== -->
-  <xacro:property name="barrel_radius" value="0.05"/>
-  <xacro:property name="barrel_height" value="0.12"/>
+  <xacro:property name="barrel_radius" value="0.06"/>
+  <xacro:property name="barrel_height" value="0.15"/>
+  <xacro:property name="barrel_bottom_clearance" value="0.006"/>
   <xacro:property name="barrel_mass" value="0.3"/>
   <!-- y 方向偏移（左右两侧） -->
-  <xacro:property name="barrel_y_offset" value="${chassis_width / 2.0 - 0.02}"/>
+  <xacro:property name="barrel_y_offset" value="0.110"/>
   <xacro:macro name="barrel" params="name y_sign">
     <link name="${name}">
@@ -38,5 +39,5 @@
       <parent link="base_link"/>
       <child link="${name}"/>
-      <origin xyz="0 ${y_sign * barrel_y_offset} ${chassis_height / 2.0 + barrel_height / 2.0}"
+      <origin xyz="0 ${y_sign * barrel_y_offset} ${-chassis_height / 2.0 + barrel_bottom_clearance + barrel_height / 2.0}"
               rpy="0 0 0"/>
     </joint>

File: src/robot_description/urdf/model/robot.camera.xacro (robot description, xacro)
@@ -3,16 +3,20 @@
   <!-- ========== 相机支架属性 ========== -->
   <xacro:property name="camera_bracket_length" value="0.020"/>
-  <xacro:property name="camera_bracket_width" value="0.040"/>
-  <xacro:property name="camera_bracket_height" value="0.015"/>
+  <xacro:property name="camera_bracket_width" value="0.0042"/>
+  <xacro:property name="camera_bracket_height" value="0.0482060266977644"/>
+  <xacro:property name="camera_bracket_mount_length" value="0.0357060266977644"/>
+  <xacro:property name="camera_bracket_origin_y" value="0.0116030133488822"/>
   <xacro:property name="camera_bracket_mass" value="0.02"/>
   <!-- ========== 相机属性 ========== -->
-  <xacro:property name="camera_box_size" value="0.025"/>
+  <xacro:property name="camera_box_length" value="0.025"/>
+  <xacro:property name="camera_box_width" value="0.090"/>
+  <xacro:property name="camera_box_height" value="0.025"/>
   <xacro:property name="camera_mass" value="0.03"/>
   <!-- ========== 相机支架链接 ========== -->
   <link name="camera_bracket">
     <visual>
-      <origin xyz="0 0 0" rpy="0 0 0"/>
+      <origin xyz="0 ${camera_bracket_origin_y} 0" rpy="0 0 0"/>
       <geometry>
-        <box size="${camera_bracket_length} ${camera_bracket_width} ${camera_bracket_height}"/>
+        <box size="${camera_bracket_length} ${camera_bracket_height} ${camera_bracket_width}"/>
       </geometry>
       <material name="black">
@@ -21,31 +25,30 @@
     </visual>
     <collision>
-      <origin xyz="0 0 0" rpy="0 0 0"/>
+      <origin xyz="0 ${camera_bracket_origin_y} 0" rpy="0 0 0"/>
       <geometry>
-        <box size="${camera_bracket_length} ${camera_bracket_width} ${camera_bracket_height}"/>
+        <box size="${camera_bracket_length} ${camera_bracket_height} ${camera_bracket_width}"/>
       </geometry>
     </collision>
     <inertial>
-      <origin xyz="0 0 0" rpy="0 0 0"/>
+      <origin xyz="0 ${camera_bracket_origin_y} 0" rpy="0 0 0"/>
       <mass value="${camera_bracket_mass}"/>
-      <inertia ixx="${camera_bracket_mass / 12.0 * (camera_bracket_width**2 + camera_bracket_height**2)}"
+      <inertia ixx="${camera_bracket_mass / 12.0 * (camera_bracket_height**2 + camera_bracket_width**2)}"
                ixy="0" ixz="0"
-               iyy="${camera_bracket_mass / 12.0 * (camera_bracket_length**2 + camera_bracket_height**2)}"
+               iyy="${camera_bracket_mass / 12.0 * (camera_bracket_length**2 + camera_bracket_width**2)}"
                iyz="0"
-               izz="${camera_bracket_mass / 12.0 * (camera_bracket_length**2 + camera_bracket_width**2)}"/>
+               izz="${camera_bracket_mass / 12.0 * (camera_bracket_length**2 + camera_bracket_height**2)}"/>
     </inertial>
   </link>
-  <!-- 支架固定在 arm_link4 基部侧面 -->
   <joint name="camera_bracket_joint" type="fixed">
-    <parent link="arm_link4"/>
+    <parent link="arm_link3"/>
     <child link="camera_bracket"/>
-    <origin xyz="${-gripper_base_length/2 - camera_bracket_height/2} 0 0" rpy="0 ${-PI/2} 0"/>
+    <origin xyz="-0.0507060266977644 0 0.0505384841187764" rpy="0 0 ${-PI/2}"/>
   </joint>
   <!-- ========== 相机链接 ========== -->
   <link name="camera_link">
     <visual>
-      <origin xyz="0 0 0" rpy="0 0 0"/>
+      <origin xyz="0 -0.032 0" rpy="0 0 0"/>
       <geometry>
-        <box size="${camera_box_size} ${camera_box_size} ${camera_box_size}"/>
+        <box size="${camera_box_length} ${camera_box_width} ${camera_box_height}"/>
       </geometry>
       <material name="grey">
@@ -54,17 +57,17 @@
     </visual>
     <collision>
-      <origin xyz="0 0 0" rpy="0 0 0"/>
+      <origin xyz="0 -0.032 0" rpy="0 0 0"/>
       <geometry>
-        <box size="${camera_box_size} ${camera_box_size} ${camera_box_size}"/>
+        <box size="${camera_box_length} ${camera_box_width} ${camera_box_height}"/>
       </geometry>
     </collision>
     <inertial>
-      <origin xyz="0 0 0" rpy="0 0 0"/>
+      <origin xyz="0 -0.032 0" rpy="0 0 0"/>
       <mass value="${camera_mass}"/>
-      <inertia ixx="${camera_mass / 12.0 * (camera_box_size**2 + camera_box_size**2)}"
+      <inertia ixx="${camera_mass / 12.0 * (camera_box_width**2 + camera_box_height**2)}"
                ixy="0" ixz="0"
-               iyy="${camera_mass / 12.0 * (camera_box_size**2 + camera_box_size**2)}"
+               iyy="${camera_mass / 12.0 * (camera_box_length**2 + camera_box_height**2)}"
                iyz="0"
-               izz="${camera_mass / 12.0 * (camera_box_size**2 + camera_box_size**2)}"/>
+               izz="${camera_mass / 12.0 * (camera_box_length**2 + camera_box_width**2)}"/>
     </inertial>
   </link>
@@ -73,5 +76,5 @@
     <parent link="camera_bracket"/>
     <child link="camera_link"/>
-    <origin xyz="0 0 ${camera_bracket_height/2 + camera_box_size/2}" rpy="0 0 0"/>
+    <origin xyz="-0.032 0 0.014475" rpy="${PI} ${-PI/2} ${-PI/2}"/>
   </joint>
   <!-- ========== 相机光学坐标框架 (ROS 相机惯例) ========== -->

File: src/robot_description/urdf/model/robot.lidar.xacro (robot description, xacro)
@@ -8,5 +8,5 @@
   <!-- ========== 支架属性 ========== -->
   <xacro:property name="bracket_radius" value="0.015"/>
-  <xacro:property name="bracket_height" value="0.35"/>
+  <xacro:property name="bracket_height" value="0.318"/>
   <xacro:property name="bracket_mass" value="0.02"/>
   <!-- ========== 支架链接 ========== -->
@@ -41,5 +41,5 @@
     <parent link="base_link"/>
     <child link="lidar_bracket"/>
-    <origin xyz="${-(chassis_length/2 - 0.05)} 0 ${chassis_height/2 + bracket_height/2}" rpy="0 0 0"/>
+    <origin xyz="${-(chassis_length/2 - 0.055)} 0 ${chassis_height/2 + bracket_height/2}" rpy="0 0 0"/>
   </joint>
   <!-- ========== 激光雷达传感器链接 ========== -->

File: src/robot_description/urdf/model/robot.model.xacro (robot description, xacro)
@@ -5,15 +5,16 @@
   <xacro:property name="PI" value="3.1415926535897931"/>
   <!-- 底盘属性 -->
-  <xacro:property name="chassis_length" value="0.300"/>
-  <xacro:property name="chassis_width" value="0.200"/>
-  <xacro:property name="chassis_height" value="0.050"/>
+  <xacro:property name="chassis_length" value="0.370"/>
+  <xacro:property name="chassis_width" value="0.270"/>
+  <xacro:property name="chassis_height" value="0.071"/>
   <xacro:property name="chassis_mass" value="5.0"/>
   <!-- 轮子属性 -->
-  <xacro:property name="wheel_radius" value="0.030"/>
-  <xacro:property name="wheel_thickness" value="0.025"/>
+  <xacro:property name="wheel_radius" value="0.04175"/>
+  <xacro:property name="wheel_thickness" value="0.033"/>
   <xacro:property name="wheel_mass" value="0.5"/>
   <!-- 安装位置偏移 -->
-  <xacro:property name="wheel_z_offset" value="0.030"/>
-  <xacro:property name="wheel_x_offset" value="0.100"/>
+  <xacro:property name="wheel_z_offset" value="0.06975"/>
+  <xacro:property name="wheel_x_offset" value="0.138"/>
+  <xacro:property name="wheel_y_offset" value="0.162"/>
   <!-- ========== 底盘 ========== -->
   <xacro:include filename="robot.chassis.xacro"/>

File: src/robot_description/urdf/model/robot.wheels.xacro (robot description, xacro)
@@ -32,5 +32,5 @@
       <parent link="base_link"/>
       <child link="${name}"/>
-      <origin xyz="${x_sign * wheel_x_offset} ${y_sign * (chassis_width/2 + wheel_thickness/2)} ${-wheel_z_offset}" rpy="0 0 0"/>
+      <origin xyz="${x_sign * wheel_x_offset} ${y_sign * wheel_y_offset} ${-wheel_z_offset}" rpy="0 0 0"/>
       <axis xyz="0 1 0"/>
     </joint>
